File: PCB/adc_board/adc_with_amps.sch (KiCad schematic (older format))
At the start: 5 parts, among them U3 MCP3564-E_ST

Commit message: Finished layout for adc board
Parts:
- added TP17: 3V3_REF, TestPoint:TestPoint_Pad_D1.0mm, symbol Connector:TestPoint
- added TP18: AVDD, TestPoint:TestPoint_Pad_D1.0mm, symbol Connector:TestPoint
- added TP19, TP21: GND, TestPoint:TestPoint_Pad_D1.0mm, symbol Connector:TestPoint
- added TP20: DVDD, TestPoint:TestPoint_Pad_D1.0mm, symbol Connector:TestPoint
- added TP22: CLK, TestPoint:TestPoint_Pad_D1.0mm, symbol Connector:TestPoint
- added TP23: MISO, TestPoint:TestPoint_Pad_D1.0mm, symbol Connector:TestPoint
- added TP24: MOSI, TestPoint:TestPoint_Pad_D1.0mm, symbol Connector:TestPoint
- added TP25: SCK, TestPoint:TestPoint_Pad_D1.0mm, symbol Connector:TestPoint
- added TP26: CS, TestPoint:TestPoint_Pad_D1.0mm, symbol Connector:TestPoint
- added TP27: IRQ, TestPoint:TestPoint_Pad_D1.0mm, symbol Connector:TestPoint
Connections:
- net 3V3_REF: now also TP17.1
- net ADC_CLK: now also TP22.1
- net ADC_IRQ*: now also TP27.1
- net AVDD: now also TP18.1
- net DVDD: now also TP20.1
- net GND: now also TP19.1, TP21.1
- net SPI_CS*: now also TP26.1
- net SPI_MISO: now also TP23.1
- net SPI_MOSI: now also TP24.1
- net SPI_SCK: now also TP25.1
Changed lines of the file:
@@
 ADC_CH7
 $Comp
-L power:GND #PWR021
+L power:GND #PWR028
 U 1 1 61579E69
 P 2600 2200
-F 0 "#PWR021" H 2600 1950 50  0001 C CNN
+F 0 "#PWR028" H 2600 1950 50  0001 C CNN
 F 1 "GND" H 2605 2027 50  0000 C CNN
 F 2 "" H 2600 2200 50  0001 C CNN
@@
 $EndComp
 $Comp
-L power:GND #PWR023
+L power:GND #PWR031
 U 1 1 6157A217
 P 3400 2100
-F 0 "#PWR023" H 3400 1850 50  0001 C CNN
+F 0 "#PWR031" H 3400 1850 50  0001 C CNN
 F 1 "GND" H 3405 1927 50  0000 C CNN
 F 2 "" H 3400 2100 50  0001 C CNN
@@
 $EndComp
 $Comp
-L power:GND #PWR024
+L power:GND #PWR032
 U 1 1 6157A41D
 P 7300 2100
-F 0 "#PWR024" H 7300 1850 50  0001 C CNN
+F 0 "#PWR032" H 7300 1850 50  0001 C CNN
 F 1 "GND" H 7305 1927 50  0000 C CNN
 F 2 "" H 7300 2100 50  0001 C CNN
@@
 $EndComp
 $Comp
-L power:GND #PWR026
+L power:GND #PWR035
 U 1 1 6157A8D7
 P 7900 2200
-F 0 "#PWR026" H 7900 1950 50  0001 C CNN
+F 0 "#PWR035" H 7900 1950 50  0001 C CNN
 F 1 "GND" H 7905 2027 50  0000 C CNN
 F 2 "" H 7900 2200 50  0001 C CNN
@@
 	7500 2000 7900 2000
 $Comp
-L power:GND #PWR025
+L power:GND #PWR033
 U 1 1 61595279
 P 7500 2200
-F 0 "#PWR025" H 7500 1950 50  0001 C CNN
+F 0 "#PWR033" H 7500 1950 50  0001 C CNN
 F 1 "GND" H 7505 2027 50  0000 C CNN
 F 2 "" H 7500 2200 50  0001 C CNN
@@
 	1    0    0    -1
 $EndComp
-Wire Wire Line
-	6800 2000 7500 2000
-$Comp
-L power:GND #PWR022
+$Comp
+L power:GND #PWR029
 U 1 1 6159B05E
 P 3000 2200
-F 0 "#PWR022" H 3000 1950 50  0001 C CNN
+F 0 "#PWR029" H 3000 1950 50  0001 C CNN
 F 1 "GND" H 3005 2027 50  0000 C CNN
 F 2 "" H 3000 2200 50  0001 C CNN
@@
 Wire Wire Line
 	4150 2300 4600 2300
+$Comp
+L Connector:TestPoint TP?
+U 1 1 61A9A0F5
+P 8900 2800
+AR Path="/61550FD5/6192F677/61A9A0F5" Ref="TP?"  Part="1"
+AR Path="/61550FD5/61994748/61A9A0F5" Ref="TP?"  Part="1"
+AR Path="/61550FD5/6199965E/61A9A0F5" Ref="TP?"  Part="1"
+AR Path="/61550FD5/6199B12D/61A9A0F5" Ref="TP?"  Part="1"
+AR Path="/61550FD5/61A9A0F5" Ref="TP23"  Part="1"
+F 0 "TP23" H 8842 2826 50  0000 R CNN
+F 1 "MISO" H 8842 2917 50  0000 R CNN
+F 2 "TestPoint:TestPoint_Pad_D1.0mm" H 9100 2800 50  0001 C CNN
+F 3 "~" H 9100 2800 50  0001 C CNN
+	1    8900 2800
+	-1   0    0    1
+$EndComp
+Text HLabel 8900 2800 1    50   Input ~ 0
+SPI_MISO
+$Comp
+L Connector:TestPoint TP?
+U 1 1 61A9ADDD
+P 9200 2800
+AR Path="/61550FD5/6192F677/61A9ADDD" Ref="TP?"  Part="1"
+AR Path="/61550FD5/61994748/61A9ADDD" Ref="TP?"  Part="1"
+AR Path="/61550FD5/6199965E/61A9ADDD" Ref="TP?"  Part="1"
+AR Path="/61550FD5/6199B12D/61A9ADDD" Ref="TP?"  Part="1"
+AR Path="/61550FD5/61A9ADDD" Ref="TP24"  Part="1"
+F 0 "TP24" H 9142 2826 50  0000 R CNN
+F 1 "MOSI" H 9142 2917 50  0000 R CNN
+F 2 "TestPoint:TestPoint_Pad_D1.0mm" H 9400 2800 50  0001 C CNN
+F 3 "~" H 9400 2800 50  0001 C CNN
+	1    9200 2800
+	-1   0    0    1
+$EndComp
+$Comp
+L Connector:TestPoint TP?
+U 1 1 61A9B2B5
+P 9500 2800
+AR Path="/61550FD5/6192F677/61A9B2B5" Ref="TP?"  Part="1"
+AR Path="/61550FD5/61994748/61A9B2B5" Ref="TP?"  Part="1"
+AR Path="/61550FD5/6199965E/61A9B2B5" Ref="TP?"  Part="1"
+AR Path="/61550FD5/6199B12D/61A9B2B5" Ref="TP?"  Part="1"
+AR Path="/61550FD5/61A9B2B5" Ref="TP25"  Part="1"
+F 0 "TP25" H 9442 2826 50  0000 R CNN
+F 1 "SCK" H 9442 2917 50  0000 R CNN
+F 2 "TestPoint:TestPoint_Pad_D1.0mm" H 9700 2800 50  0001 C CNN
+F 3 "~" H 9700 2800 50  0001 C CNN
+	1    9500 2800
+	-1   0    0    1
+$EndComp
+$Comp
+L Connector:TestPoint TP?
+U 1 1 61A9B73D
+P 9800 2800
+AR Path="/61550FD5/6192F677/61A9B73D" Ref="TP?"  Part="1"
+AR Path="/61550FD5/61994748/61A9B73D" Ref="TP?"  Part="1"
+AR Path="/61550FD5/6199965E/61A9B73D" Ref="TP?"  Part="1"
+AR Path="/61550FD5/6199B12D/61A9B73D" Ref="TP?"  Part="1"
+AR Path="/61550FD5/61A9B73D" Ref="TP26"  Part="1"
+F 0 "TP26" H 9742 2826 50  0000 R CNN
+F 1 "CS" H 9742 2917 50  0000 R CNN
+F 2 "TestPoint:TestPoint_Pad_D1.0mm" H 10000 2800 50  0001 C CNN
+F 3 "~" H 10000 2800 50  0001 C CNN
+	1    9800 2800
+	-1   0    0    1
+$EndComp
+Text HLabel 9200 2800 1    50   Input ~ 0
+SPI_MOSI
+Text HLabel 9500 2800 1    50   Input ~ 0
+SPI_SCK
+Text HLabel 9800 2800 1    50   Input ~ 0
+SPI_CS*
+Text HLabel 10050 2800 1    50   Input ~ 0
+ADC_IRQ*
+$Comp
+L Connector:TestPoint TP?
+U 1 1 61AA16B1
+P 10050 2800
+AR Path="/61550FD5/6192F677/61AA16B1" Ref="TP?"  Part="1"
+AR Path="/61550FD5/61994748/61AA16B1" Ref="TP?"  Part="1"
+AR Path="/61550FD5/6199965E/61AA16B1" Ref="TP?"  Part="1"
+AR Path="/61550FD5/6199B12D/61AA16B1" Ref="TP?"  Part="1"
+AR Path="/61550FD5/61AA16B1" Ref="TP27"  Part="1"
+F 0 "TP27" H 9992 2826 50  0000 R CNN
+F 1 "IRQ" H 9992 2917 50  0000 R CNN
+F 2 "TestPoint:TestPoint_Pad_D1.0mm" H 10250 2800 50  0001 C CNN
+F 3 "~" H 10250 2800 50  0001 C CNN
+	1    10050 2800
+	-1   0    0    1
+$EndComp
+Text HLabel 8600 2800 1    50   Input ~ 0
+ADC_CLK
+$Comp
+L Connector:TestPoint TP?
+U 1 1 61A9E5D5
+P 8600 2800
+AR Path="/61550FD5/6192F677/61A9E5D5" Ref="TP?"  Part="1"
+AR Path="/61550FD5/61994748/61A9E5D5" Ref="TP?"  Part="1"
+AR Path="/61550FD5/6199965E/61A9E5D5" Ref="TP?"  Part="1"
+AR Path="/61550FD5/6199B12D/61A9E5D5" Ref="TP?"  Part="1"
+AR Path="/61550FD5/61A9E5D5" Ref="TP22"  Part="1"
+F 0 "TP22" H 8542 2826 50  0000 R CNN
+F 1 "CLK" H 8542 2917 50  0000 R CNN
+F 2 "TestPoint:TestPoint_Pad_D1.0mm" H 8800 2800 50  0001 C CNN
+F 3 "~" H 8800 2800 50  0001 C CNN
+	1    8600 2800
+	-1   0    0    1
+$EndComp
+Wire Wire Line
+	6800 2000 7500 2000
+$Comp
+L Connector:TestPoint TP?
+U 1 1 61AAE3E8
+P 7300 1400
+AR Path="/61550FD5/6192F677/61AAE3E8" Ref="TP?"  Part="1"
+AR Path="/61550FD5/61994748/61AAE3E8" Ref="TP?"  Part="1"
+AR Path="/61550FD5/6199965E/61AAE3E8" Ref="TP?"  Part="1"
+AR Path="/61550FD5/6199B12D/61AAE3E8" Ref="TP?"  Part="1"
+AR Path="/61550FD5/61AAE3E8" Ref="TP20"  Part="1"
+F 0 "TP20" H 7242 1426 50  0000 R CNN
+F 1 "DVDD" H 7242 1517 50  0000 R CNN
+F 2 "TestPoint:TestPoint_Pad_D1.0mm" H 7500 1400 50  0001 C CNN
+F 3 "~" H 7500 1400 50  0001 C CNN
+	1    7300 1400
+	-1   0    0    1
+$EndComp
+$Comp
+L Connector:TestPoint TP?
+U 1 1 61AAE78D
+P 7600 1400
+AR Path="/61550FD5/6192F677/61AAE78D" Ref="TP?"  Part="1"
+AR Path="/61550FD5/61994748/61AAE78D" Ref="TP?"  Part="1"
+AR Path="/61550FD5/6199965E/61AAE78D" Ref="TP?"  Part="1"
+AR Path="/61550FD5/6199B12D/61AAE78D" Ref="TP?"  Part="1"
+AR Path="/61550FD5/61AAE78D" Ref="TP21"  Part="1"
+F 0 "TP21" H 7542 1426 50  0000 R CNN
+F 1 "GND" H 7542 1517 50  0000 R CNN
+F 2 "TestPoint:TestPoint_Pad_D1.0mm" H 7800 1400 50  0001 C CNN
+F 3 "~" H 7800 1400 50  0001 C CNN
+	1    7600 1400
+	-1   0    0    1
+$EndComp
+Text HLabel 7300 1400 1    50   Input ~ 0
+DVDD
+$Comp
+L power:GND #PWR034
+U 1 1 61AAEFD9
+P 7600 1400
+F 0 "#PWR034" H 7600 1150 50  0001 C CNN
+F 1 "GND" H 7605 1227 50  0000 C CNN
+F 2 "" H 7600 1400 50  0001 C CNN
+F 3 "" H 7600 1400 50  0001 C CNN
+	1    7600 1400
+	-1   0    0    1
+$EndComp
+$Comp
+L Connector:TestPoint TP?
+U 1 1 61AB5425
+P 3150 1400
+AR Path="/61550FD5/6192F677/61AB5425" Ref="TP?"  Part="1"
+AR Path="/61550FD5/61994748/61AB5425" Ref="TP?"  Part="1"
+AR Path="/61550FD5/6199965E/61AB5425" Ref="TP?"  Part="1"
+AR Path="/61550FD5/6199B12D/61AB5425" Ref="TP?"  Part="1"
+AR Path="/61550FD5/61AB5425" Ref="TP19"  Part="1"
+F 0 "TP19" H 3092 1426 50  0000 R CNN
+F 1 "GND" H 3092 1517 50  0000 R CNN
+F 2 "TestPoint:TestPoint_Pad_D1.0mm" H 3350 1400 50  0001 C CNN
+F 3 "~" H 3350 1400 50  0001 C CNN
+	1    3150 1400
+	-1   0    0    1
+$EndComp
+$Comp
+L power:GND #PWR030
+U 1 1 61AB542C
+P 3150 1400
+F 0 "#PWR030" H 3150 1150 50  0001 C CNN
+F 1 "GND" H 3155 1227 50  0000 C CNN
+F 2 "" H 3150 1400 50  0001 C CNN
+F 3 "" H 3150 1400 50  0001 C CNN
+	1    3150 1400
+	-1   0    0    1
+$EndComp
+Text HLabel 2850 1400 1    50   Input ~ 0
+AVDD
+$Comp
+L Connector:TestPoint TP?
+U 1 1 61ABB068
+P 2400 1400
+AR Path="/61550FD5/6192F677/61ABB068" Ref="TP?"  Part="1"
+AR Path="/61550FD5/61994748/61ABB068" Ref="TP?"  Part="1"
+AR Path="/61550FD5/6199965E/61ABB068" Ref="TP?"  Part="1"
+AR Path="/61550FD5/6199B12D/61ABB068" Ref="TP?"  Part="1"
+AR Path="/61550FD5/61ABB068" Ref="TP17"  Part="1"
+F 0 "TP17" H 2342 1426 50  0000 R CNN
+F 1 "3V3_REF" H 2342 1517 50  0000 R CNN
+F 2 "TestPoint:TestPoint_Pad_D1.0mm" H 2600 1400 50  0001 C CNN
+F 3 "~" H 2600 1400 50  0001 C CNN
+	1    2400 1400
+	-1   0    0    1
+$EndComp
+Text HLabel 2400 1400 1    50   Input ~ 0
+3V3_REF
+$Comp
+L Connector:TestPoint TP?
+U 1 1 61AB541F
+P 2850 1400
+AR Path="/61550FD5/6192F677/61AB541F" Ref="TP?"  Part="1"
+AR Path="/61550FD5/61994748/61AB541F" Ref="TP?"  Part="1"
+AR Path="/61550FD5/6199965E/61AB541F" Ref="TP?"  Part="1"
+AR Path="/61550FD5/6199B12D/61AB541F" Ref="TP?"  Part="1"
+AR Path="/61550FD5/61AB541F" Ref="TP18"  Part="1"
+F 0 "TP18" H 2792 1426 50  0000 R CNN
+F 1 "AVDD" H 2792 1517 50  0000 R CNN
+F 2 "TestPoint:TestPoint_Pad_D1.0mm" H 3050 1400 50  0001 C CNN
+F 3 "~" H 3050 1400 50  0001 C CNN
+	1    2850 1400
+	-1   0    0    1
+$EndComp
 $EndSCHEMATC
