File: PCB/bridge_board/bridge_board.sch (KiCad schematic (older format))
At the start: 9 parts, among them J1 54-00177, J2 1702473

Commit message: Finished layout for adc board
Parts:
- J1: symbol 54-00177:54-00177 -> bridge_board-rescue:54-00177-54-00177
Changed lines of the file:
@@
 $EndDescr
 $Comp
-L 54-00177:54-00177 J1
+L bridge_board-rescue:54-00177-54-00177 J1
 U 1 1 612B7BBF
 P 3800 3650
