File: PCB/main_board/main_board.kicad_pcb (KiCad board)
At the start: 4 copper layers, 122 parts, among them J1 Conn_01x13, J10 54-00177, J11 54-00177, J12 54-00177, J13 54-00177, J14 54-00177, J2 TSM-107-01-T-SV, J3 54-00177, J4 54-00177, J5 54-00177, J6 54-00177, J7 54-00177, J8 54-00177, J9 54-00177, U1 Pico, U10 MAX4209HAUA, U11 MAX4209HAUA, U12 MAX4209HAUA, U13 MAX4209HAUA, U14 MCP3564-E_ST, U15 MAX4209HAUA, U16 MAX4209HAUA, U17 MAX4209HAUA, U18 MAX4209HAUA, U2 MAX6070BAUT33T, U3 TPS62046DGQR, U4 MCP3564-E_ST, U5 MAX4209HAUA, U6 MAX4209HAUA, U7 MAX4209HAUA, U8 MAX4209HAUA, U9 MCP3564-E_ST

Commit message: Adding gerbers, and updated version of main board
Parts:
- removed C1, C4, C6, C7, C8: 10uF, Capacitor_SMD:C_0805_2012Metric_Pad1.18x1.45mm_HandSolder
- removed C10, C12, C13, C14, C16, C17, C18, C2, C20, C21, C22, C24, C25, C26, C27, C28, C3, C30, C31, C32, C34, C35, C36, C38, C39, C40, C42, C43, C44, C45, C46, C48, C49, C5, C50, C52, C53, C54, C56, C57, C58, C60, C61, C62, C9: 0.1uF, Capacitor_SMD:C_0805_2012Metric_Pad1.18x1.45mm_HandSolder
- removed C11, C15, C19, C23, C29, C33, C37, C41, C47, C51, C55, C59: 10nF, Capacitor_SMD:C_0805_2012Metric_Pad1.18x1.45mm_HandSolder
- removed J10, J11, J12, J13, J14, J7, J8, J9: 54-00177, 54-00177:54-00177
- removed L1: 6.2uH, 744062006:744062006
- removed NT1: Net-Tie_2, NetTie:NetTie-2_SMD_Pad2.0mm
- removed R1, R2: 10K, Resistor_SMD:R_0805_2012Metric_Pad1.20x1.40mm_HandSolder
- removed R10, R11, R12, R13, R14, R15, R16, R17, R18, R19, R20, R21, R22, R23, R24, R25, R26, R3, R4, R5, R6, R7, R8, R9: 100R, Resistor_SMD:R_0805_2012Metric_Pad1.20x1.40mm_HandSolder
- removed U10, U11, U12, U13, U15, U16, U17, U18, U5, U6, U7, U8: MAX4209HAUA, MAX4209HAUA:SOP65P490X110-8N
- removed U14, U4, U9: MCP3564-E_ST, ‎MCP3564-E-ST:MCP3564-E&slash_ST
- removed U2: MAX6070BAUT33T, MAX6070BAUT33T:SOT95P280X145-6N
- removed U3: TPS62046DGQR, TPS62046DGQR:IC_XTR111AIDGQR
- added H1: MountingHole_Pad, MountingHole:MountingHole_3.2mm_M3_Pad_Via, F.Cu at (157.5, 83.8)
- added H2: MountingHole_Pad, MountingHole:MountingHole_3.2mm_M3_Pad_Via, F.Cu at (200.7, 83.8)
- added H3: MountingHole_Pad, MountingHole:MountingHole_3.2mm_M3_Pad_Via, F.Cu at (242.6, 83.8)
- added H4: MountingHole_Pad, MountingHole:MountingHole_3.2mm_M3_Pad_Via, F.Cu at (242.6, 30.5)
- J1: footprint wifi_connector:PinHeader_1x13_P2.54mm_Vertical_SMD_Pin1Left -> wifi_connector:PinHeader_1x13_P2.54mm_Vertical_SMD_Pin1Left_with_holes
- J3, J4, J5, J6: value 54-00177 -> Conn_02x05_Counter_Clockwise; footprint 54-00177:54-00177 -> 2x5header:PinHeader_2x05_P2.54mm_Vertical_SMD
- moved J3 103.5 mm to (161.3, 71.1), turned to 0 degrees
- moved J4 93.0 mm to (181.6, 80.0), turned to 90 degrees
- moved J2 69.7 mm to (231.1, 36.8)
- moved J5 68.1 mm to (229.9, 80.0), turned to 90 degrees
- moved U1 24.2 mm to (208.3, 52.1)
- moved J6 22.7 mm to (238.4, 58.4)
- moved J1 20.0 mm to (180.3, 44.5)
Connections:
- net /CS4 renamed Net-(U1-Pad7)
- net /SPI1_MISO renamed /WIFI_MISO
- net /SPI1_MOSI renamed /WIFI_MOSI
- net /SPI1_SCK renamed /WIFI_SCK
- net Net-(J1-Pad11) renamed /NC_WIFI_CFG
- net Net-(J1-Pad12) renamed /NC_WIFI_RXD
- net Net-(J1-Pad13) renamed /NC_WIFI_TXD
- J1 pad 1: /PICO_3V3 -> +3V3
- J1 pad 2: GNDD -> GND
- J3 pad 1: +3V3 -> GND
- J3 pad 2: GNDA -> +5V
- J3 pad 3: /ADC0/Bridge1/BRIDGE+ -> /ADC0_ENABLE
- J3 pad 4: /ADC0/Bridge1/BRIDGE- -> /ADC0_PGOOD
- J3 pad 5: Net-(J3-Pad5) -> /ADC_CLK
- J3 pad 6: Net-(J3-Pad6) -> /ADC_MISO
- J4 pad 1: +3V3 -> GND
- J4 pad 2: GNDA -> +5V
- J4 pad 3: /ADC0/Bridge2/BRIDGE+ -> /ADC1_ENABLE
- J4 pad 4: /ADC0/Bridge2/BRIDGE- -> /ADC1_PGOOD
- J4 pad 5: Net-(J4-Pad5) -> /ADC_CLK
- J4 pad 6: Net-(J4-Pad6) -> /ADC_MISO
- J5 pad 1: +3V3 -> GND
- J5 pad 2: GNDA -> +5V
- J5 pad 3: /ADC0/Bridge3/BRIDGE+ -> /ADC2_ENABLE
- J5 pad 4: /ADC0/Bridge3/BRIDGE- -> /ADC2_PGOOD
- J5 pad 5: Net-(J5-Pad5) -> /ADC_CLK
- J5 pad 6: Net-(J5-Pad6) -> /ADC_MISO
- J6 pad 1: +3V3 -> GND
- J6 pad 2: GNDA -> +5V
- J6 pad 3: /ADC0/Bridge0/BRIDGE+ -> /ADC3_ENABLE
- J6 pad 4: /ADC0/Bridge0/BRIDGE- -> /ADC3_PGOOD
- J6 pad 5: Net-(J6-Pad5) -> /ADC_CLK
- J6 pad 6: Net-(J6-Pad6) -> /ADC_MISO
- U1 pad 10: /CS3 -> /ADC1_PGOOD
- U1 pad 11: /CS2 -> /ADC1_ENABLE
- U1 pad 12: /WIFI_EN -> /WIFI_RST
- U1 pad 13: GNDD -> GND
- U1 pad 18: GNDD -> GND
- U1 pad 19: /WIFI_RST -> /WIFI_EN
- U1 pad 21: /SPI0_MISO -> /ADC_MISO
- U1 pad 22: /CS0 -> /ADC2_CS
- U1 pad 23: GNDD -> GND
- U1 pad 24: /SPI0_SCK -> /ADC_SCK
- U1 pad 25: /SPI0_MOSI -> /ADC_MOSI
- U1 pad 26: Net-(U1-Pad26) -> /ADC2_PGOOD
- U1 pad 27: Net-(U1-Pad27) -> /ADC2_ENABLE
- U1 pad 28: GNDD -> GND
- U1 pad 3: GNDD -> GND
- U1 pad 31: Net-(U1-Pad31) -> /ADC3_CS
- U1 pad 32: Net-(U1-Pad32) -> /ADC3_PGOOD
- U1 pad 33: GNDD -> GND
- U1 pad 34: /CS1 -> /ADC3_ENABLE
- U1 pad 36: /PICO_3V3 -> +3V3
- U1 pad 38: GNDD -> GND
- U1 pad 4: /CS7 -> /ADC0_CS
- U1 pad 42: GNDD -> GND
- U1 pad 5: /CS6 -> /ADC0_PGOOD
- U1 pad 6: /CS5 -> /ADC0_ENABLE
- U1 pad 8: GNDD -> GND
- U1 pad 9: Net-(U1-Pad9) -> /ADC1_CS
Routing:
- net +3V3: track 785.5 -> 3.22 mm, vias 25 -> 0
- net GNDA: track 760.5 -> 0.00 mm, vias 71 -> 0
- net GNDD: track 481.0 -> 0.00 mm, vias 19 -> 0
- net /1V65_REF: track 214.4 -> 0.00 mm, vias 13 -> 0
- net /ADC_MOSI: track 0.00 -> 118.0 mm, vias 0 -> 7
- net /ADC_SCK: track 0.00 -> 111.8 mm, vias 0 -> 3
- net /ADC_MISO: track 0.00 -> 109.6 mm, vias 0 -> 7
- net /PICO_3V3: track 109.2 -> 0.00 mm, vias 6 -> 0
- net /3V3_REF_OUT: track 96.5 -> 0.00 mm, vias 4 -> 0
- net /ADC_CLK: track 61.0 -> 136.1 mm, vias 2 -> 7
- net /SPI0_MISO: track 72.1 -> 0.00 mm, vias 4 -> 0
- net /ADC0_PGOOD: track 0.00 -> 61.0 mm, vias 0 -> 2
- net +5V: track 61.4 -> 1.35 mm
- net /ADC0_ENABLE: track 0.00 -> 55.5 mm, vias 0 -> 2
- net /SPI0_SCK: track 55.0 -> 0.00 mm, vias 4 -> 0
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- added copper zone on F.Cu, net +3V3
- added copper zone on F.Cu, net +5V
- added copper zone on B.Cu, net GND
Other:
- board outline added: 95.2 x 63.5 mm
- copper layers 4 -> 2
