File: PCB/main_board/main_board.sch (KiCad schematic (older format))
At the start: 17 parts, among them J1 Conn_01x13, J2 TSM-107-01-T-SV, U1 Pico, U2 MAX6070BAUT33T, U3 TPS62046DGQR

Commit message: Adding gerbers, and updated version of main board
Parts:
- removed C1, C4, C6, C7, C8: 10uF, Capacitor_SMD:C_0805_2012Metric_Pad1.18x1.45mm_HandSolder, symbol Device:C_Small
- removed C2, C3, C5: 0.1uF, Capacitor_SMD:C_0805_2012Metric_Pad1.18x1.45mm_HandSolder, symbol Device:C_Small
- removed L1: 6.2uH, 744062006:744062006, symbol Device:L_Small
- removed NT1: Net-Tie_2, NetTie:NetTie-2_SMD_Pad2.0mm, symbol Device:Net-Tie_2
- removed R1, R2: 10K, Resistor_SMD:R_0805_2012Metric_Pad1.20x1.40mm_HandSolder, symbol Device:R_Small
- removed U2: MAX6070BAUT33T, MAX6070BAUT33T:SOT95P280X145-6N, symbol MAX6070BAUT33T:MAX6070BAUT33T
- removed U3: TPS62046DGQR, TPS62046DGQR:IC_XTR111AIDGQR, symbol TPS62046DGQR:TPS62046DGQR
- added H1, H2, H3, H4: MountingHole_Pad, MountingHole:MountingHole_3.2mm_M3_Pad_Via, symbol Mechanical:MountingHole_Pad
- J1: footprint wifi_connector:PinHeader_1x13_P2.54mm_Vertical_SMD_Pin1Left -> wifi_connector:PinHeader_1x13_P2.54mm_Vertical_SMD_Pin1Left_with_holes
Connections:
- net PICO_3V3 is gone; now on net +3V3: J1.1 (Pin_1), U1.36 (3V3)
- net SWCLK: now also J2.3 (SWCLK); no longer J2.5 (SWDIO)
- net SWDIO: now also J2.5 (SWDIO); no longer J2.3 (SWCLK)
- net WIFI_EN: now also U1.19 (GPIO14); no longer U1.12 (GPIO9)
- net WIFI_RST: now also U1.12 (GPIO9); no longer U1.19 (GPIO14)
- net ADC2_PGOOD: now reaches U1.26 (GPIO20)
- net ADC2_ENABLE: now reaches U1.27 (GPIO21)
- net ADC3_CS: now reaches U1.31 (GPIO26_ADC0)
- net ADC3_PGOOD: now reaches U1.32 (GPIO27_ADC1)
- net ADC1_CS: now reaches U1.9 (GPIO6)
- net NC_WIFI_CFG: now reaches J1.11 (Pin_11)
- net NC_WIFI_RXD: now reaches J1.12 (Pin_12)
- net NC_WIFI_TXD: now reaches J1.13 (Pin_13)
- net CS0 renamed ADC2_CS
- net CS1 renamed ADC3_ENABLE
- net CS2 renamed ADC1_ENABLE
- net CS3 renamed ADC1_PGOOD
- net CS4: no longer names the net of U1.7 (GPIO5)
- net CS5 renamed ADC0_ENABLE
- net CS6 renamed ADC0_PGOOD
- net CS7 renamed ADC0_CS
- net GNDD renamed GND
- net GND: now also H1.1, H2.1, H3.1, H4.1
- net SPI0_MISO renamed ADC_MISO
- net SPI0_MOSI renamed ADC_MOSI
- net SPI0_SCK renamed ADC_SCK
- net SPI1_MISO renamed WIFI_MISO
- net SPI1_MOSI renamed WIFI_MOSI
- net SPI1_SCK renamed WIFI_SCK
- no-connect marks 14 -> 7
Other:
- note removed: "3.3V Regulator"
- note removed: "3.3V Voltage Reference"
- moved on the sheet: J1, U1
